File: Electronics/PCB/OpetusSmpS.kicad_sch (KiCad schematic)
At the start: 62 parts, among them J2 KPJX-4S-S, J4 Screw_Terminal_01x10, SW1 SW_SPST, SW3 SW_SPST, U1 AMS1117-3.3, U2 ADIP16-Z-LC-R, U3 SN75C3243PWR, U4 ADIP16-Z-LC-R, U5 ADIP10-Z-LC-R

Commit message: Refactor code structure for improved readability and maintainability
Parts:
- removed D4: LED, Connector_PinHeader_2.54mm:PinHeader_1x02_P2.54mm_Vertical, symbol Device:LED
- removed D5: 15V, Diode_SMD:D_SMB_Handsoldering, symbol Device:D_TVS
- added D4: 15V, Diode_SMD:D_SMB_Handsoldering, symbol Device:D_TVS
- added D5: LED, Connector_PinHeader_2.54mm:PinHeader_1x02_P2.54mm_Vertical, symbol Device:LED
- R2: value 10k -> 220; footprint Resistor_SMD:R_0805_2012Metric_Pad1.20x1.40mm_HandSolder -> Resistor_SMD:R_1206_3216Metric_Pad1.30x1.75mm_HandSolder
- R5: value 220 -> 10k; footprint Resistor_SMD:R_1206_3216Metric_Pad1.30x1.75mm_HandSolder -> Resistor_SMD:R_0805_2012Metric_Pad1.20x1.40mm_HandSolder
Connections:
- net GND: now also U2.11, U4.11, U5.3, U5.5, D4.1 (A1), D5.1 (K); no longer U2.8, U4.8, U5.1, U5.9
- net RX2_IN: now also R13.2, U3.16 (ROUT4); no longer R8.2, U3.7 (RIN4)
- net RX2_OUT: now also R2.1, U3.7 (RIN4); no longer R10.1, U3.16 (ROUT4)
- net RX3_IN: now also R12.2, U3.15 (ROUT5); no longer R13.2, U3.8 (RIN5)
- net RX3_OUT: now also R22.1, U3.8 (RIN5); no longer R5.1, U3.15 (ROUT5)
- net RX_IN: now also R7.2, U3.17 (ROUT3); no longer R4.2, U3.6 (RIN3)
- net RX_OUT: now also R10.1, U3.6 (RIN3); no longer R22.1, U3.17 (ROUT3)
- net TX2_IN: now also R3.2; no longer R7.2
- net TX2_OUT: now also R1.1; no longer R6.1
- net TX3_IN: now also R4.2; no longer R12.2
- net TX3_OUT: now also R20.1; no longer R1.1
- net TX_IN: now also R8.2; no longer R3.2
- net TX_OUT: now also R6.1; no longer R20.1
- net at U4.14: no longer R5.2
- net at R2.2: now also U4.10, D4.2 (A2)
- net at U2.10: now also D21.2 (A2), R22.2
- net at D19.2 (A2), R20.2: now also U2.8; no longer U2.12
- net at U2.16: now also F2.2, R21.1
- net at U2.4: no longer U2.9
- net at D6.2 (A2), R6.2: now also U5.4; no longer U5.3
- net at D9.2 (A2), R10.2: now also U5.7; no longer U5.5
- net at D3.2 (A2), R1.2: now also U4.8; no longer U4.12
- net at U4.16: now also F3.2, R5.1
- net at U4.4: no longer U4.9
- new net: U4.12, U4.3
- new net: U2.12, U2.3
- new net: D5.2 (A), R5.2
- now unconnected: U2.14
Other:
- moved on the sheet: D19, D20, D21, D6, D9, F2, R10, R20, R21, R22, R6, U2
